File: corneds/corneds.kicad_pcb (KiCad board)
At the start: 2 copper layers, 320 x 104.9 mm, 130 parts, among them J1 Conn_ARM_SWD_TagConnect_TC203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, J2 Conn_ARM_SWD_TagConnect_TC203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, J3 AudioJack4, J4 AudioJack4, SW1 SW_Push, SW10 SW_Push, SW11 SW_Push, SW12 SW_Push, SW13 SW_Push, SW14 SW_Push, SW15 SW_Push, SW16 SW_Push, SW17 SW_Push, SW18 SW_Push, SW19 SW_Push, SW2 SW_Push, SW20 SW_Push, SW21 SW_Push, SW22 SW_Push, SW23 SW_Push, SW24 SW_Push, SW25 SW_Push, SW26 SW_Push, SW27 SW_Push, SW28 SW_Push, SW29 SW_Push, SW3 SW_Push, SW30 SW_Push, SW31 SW_Push, SW32 SW_Push, SW33 SW_Push, SW34 SW_Push, SW35 SW_Push, SW36 SW_Push, SW37 SW_Push, SW38 SW_Push, SW39 SW_Push, SW4 SW_Push, SW40 SW_Push, SW41 SW_Push, SW42 SW_Push, SW5 SW_Push, SW6 SW_Push, SW7 SW_Push, SW8 SW_Push, SW9 SW_Push, U1 Pico, U2 Pico

Commit message: ordered version
Parts:
- removed DBG1, DBG7: GND, Connector_PinSocket_2.54mm:PinSocket_1x01_P2.54mm_Vertical
- removed DBG10, DBG4: TX, Connector_PinSocket_2.54mm:PinSocket_1x01_P2.54mm_Vertical
- removed DBG11, DBG5: RX, Connector_PinSocket_2.54mm:PinSocket_1x01_P2.54mm_Vertical
- removed DBG12, DBG6: RTS, Connector_PinSocket_2.54mm:PinSocket_1x01_P2.54mm_Vertical
- removed DBG2, DBG8: CTS, Connector_PinSocket_2.54mm:PinSocket_1x01_P2.54mm_Vertical
- removed DBG3, DBG9: 5V, Connector_PinSocket_2.54mm:PinSocket_1x01_P2.54mm_Vertical
- removed J1, J2: Conn_ARM_SWD_TagConnect_TC2030-NL, Connector:Tag-Connect_TC2030-IDC-NL_2x03_P1.27mm_Vertical
- added U3: SWD_Connector_3pin, entropy:SM03B-SRSS-TB, F.Cu at (126.5, 108.8)
- added U4: SWD_Connector_3pin, entropy:SM03B-SRSS-TB, F.Cu at (163.0, 108.8)
- added U5: Debug_UART_l, entropy:Header_6pin, F.Cu at (-2.54, 104.1)
- added U6: Debug_UART_r, entropy:Header_6pin, F.Cu at (292.1, 104.1)
Routing:
- net /vcc_r: track 0.00 -> 240.4 mm, vias 0 -> 1
- net /dbg_uart_tx_r: track 0.00 -> 192.4 mm, vias 0 -> 1
- net /dbg_uart_rx_r: track 0.00 -> 191.3 mm, vias 0 -> 1
- net /xboard_uart_tx_r: track 18.1 -> 95.6 mm, vias 0 -> 1
- net /xboard_uart_rx_r: track 18.8 -> 93.8 mm
- net /swdio_l: track 28.9 -> 21.6 mm
- net /swclk_l: track 29.1 -> 22.1 mm
- net /swdio_r: track 20.4 -> 21.8 mm
- net /swclk_r: track 20.7 -> 21.6 mm
- net /gnd_l: vias 0 -> 2
- added copper zone on F.Cu, net /gnd_r
- removed copper zone on F.Cu, net (none)
Other:
- board text added: "23 Mar 2023"
- board text added: "corne"
