File: corneds/corneds.kicad_sch (KiCad schematic)
At the start: 118 parts, among them J1 Conn_ARM_SWD_TagConnect_TC203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, J2 Conn_ARM_SWD_TagConnect_TC203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, J3 AudioJack4, J4 AudioJack4, SW1 SW_Push, SW10 SW_Push, SW11 SW_Push, SW12 SW_Push, SW13 SW_Push, SW14 SW_Push, SW15 SW_Push, SW16 SW_Push, SW17 SW_Push, SW18 SW_Push, SW19 SW_Push, SW2 SW_Push, SW20 SW_Push, SW21 SW_Push, SW22 SW_Push, SW23 SW_Push, SW24 SW_Push, SW25 SW_Push, SW26 SW_Push, SW27 SW_Push, SW28 SW_Push, SW29 SW_Push, SW3 SW_Push, SW30 SW_Push, SW31 SW_Push, SW32 SW_Push, SW33 SW_Push, SW34 SW_Push, SW35 SW_Push, SW36 SW_Push, SW37 SW_Push, SW38 SW_Push, SW39 SW_Push, SW4 SW_Push, SW40 SW_Push, SW41 SW_Push, SW42 SW_Push, SW5 SW_Push, SW6 SW_Push, SW7 SW_Push, SW8 SW_Push, SW9 SW_Push, U1 Pico, U2 Pico

Commit message: finished placing left side
Parts:
- added DBG1, DBG?: GND, Connector_PinSocket_2.54mm:PinSocket_1x01_P2.54mm_Vertical, symbol Connector:TestPoint
- added DBG2, DBG?: CTS, Connector_PinSocket_2.54mm:PinSocket_1x01_P2.54mm_Vertical, symbol Connector:TestPoint
- added DBG3, DBG?: 5V, Connector_PinSocket_2.54mm:PinSocket_1x01_P2.54mm_Vertical, symbol Connector:TestPoint
- added DBG4, DBG?: TX, Connector_PinSocket_2.54mm:PinSocket_1x01_P2.54mm_Vertical, symbol Connector:TestPoint
- added DBG5, DBG?: RX, Connector_PinSocket_2.54mm:PinSocket_1x01_P2.54mm_Vertical, symbol Connector:TestPoint
- added DBG6, DBG?: RTS, Connector_PinSocket_2.54mm:PinSocket_1x01_P2.54mm_Vertical, symbol Connector:TestPoint
Connections:
- net dbg_uart_rx_l: now also DBG?.1; no longer J1.6 (SWO)
- net dbg_uart_rx_r: now also DBG5.1; no longer J2.6 (SWO)
- net dbg_uart_tx_l: now also DBG?.1; no longer J1.3 (~{RESET})
- net dbg_uart_tx_r: now also DBG4.1; no longer J2.3 (~{RESET})
- net gnd_l: now also DBG?.1
- net gnd_r: now also DBG1.1
- net vcc_l: now also DBG?.1
- net vcc_r: now also DBG3.1

Commit message: sch updates
Parts:
- gave numbers to parts that had none: 6
Changed lines of the file:
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@@
   (symbol (lib_id "Connector:TestPoint") (at 274.32 78.74 0) (unit 1)
     (in_bom yes) (on_board yes) (fields_autoplaced)
-    (property "Reference" "DBG?" (id 0) (at 276.86 74.1679 0)
+    (property "Reference" "DBG11" (id 0) (at 276.86 74.1679 0)
       (effects (font (size 1.27 1.27)) (justify left))
     )
@@
   (symbol (lib_id "Connector:TestPoint") (at 274.32 68.58 0) (unit 1)
     (in_bom yes) (on_board yes) (fields_autoplaced)
-    (property "Reference" "DBG?" (id 0) (at 276.86 64.0079 0)
+    (property "Reference" "DBG9" (id 0) (at 276.86 64.0079 0)
       (effects (font (size 1.27 1.27)) (justify left))
     )
@@
   (symbol (lib_id "Connector:TestPoint") (at 274.32 73.66 0) (unit 1)
     (in_bom yes) (on_board yes) (fields_autoplaced)
-    (property "Reference" "DBG?" (id 0) (at 276.86 69.0879 0)
+    (property "Reference" "DBG10" (id 0) (at 276.86 69.0879 0)
       (effects (font (size 1.27 1.27)) (justify left))
     )
@@
   (symbol (lib_id "Connector:TestPoint") (at 274.32 58.42 0) (unit 1)
     (in_bom yes) (on_board yes) (fields_autoplaced)
-    (property "Reference" "DBG?" (id 0) (at 276.86 53.8479 0)
+    (property "Reference" "DBG7" (id 0) (at 276.86 53.8479 0)
       (effects (font (size 1.27 1.27)) (justify left))
     )
@@
   (symbol (lib_id "Connector:TestPoint") (at 274.32 83.82 0) (unit 1)
     (in_bom yes) (on_board yes) (fields_autoplaced)
-    (property "Reference" "DBG?" (id 0) (at 276.86 79.2479 0)
+    (property "Reference" "DBG12" (id 0) (at 276.86 79.2479 0)
       (effects (font (size 1.27 1.27)) (justify left))
     )
@@
   (symbol (lib_id "Connector:TestPoint") (at 274.32 63.5 0) (unit 1)
     (in_bom yes) (on_board yes) (fields_autoplaced)
-    (property "Reference" "DBG?" (id 0) (at 276.86 58.9279 0)
+    (property "Reference" "DBG8" (id 0) (at 276.86 58.9279 0)
       (effects (font (size 1.27 1.27)) (justify left))
     )
@@
       (reference "DBG6") (unit 1) (value "RTS") (footprint "Connector_PinSocket_2.54mm:PinSocket_1x01_P2.54mm_Vertical")
     )
+    (path "/5c744d00-6e74-484c-b63b-3b58dd05dd79"
+      (reference "DBG7") (unit 1) (value "GND") (footprint "Connector_PinSocket_2.54mm:PinSocket_1x01_P2.54mm_Vertical")
+    )
+    (path "/feeb044e-58ef-4711-90fe-4a14fad0b279"
+      (reference "DBG8") (unit 1) (value "CTS") (footprint "Connector_PinSocket_2.54mm:PinSocket_1x01_P2.54mm_Vertical")
+    )
+    (path "/1a72f5d6-44ee-46ae-8a18-fbbb82588964"
+      (reference "DBG9") (unit 1) (value "5V") (footprint "Connector_PinSocket_2.54mm:PinSocket_1x01_P2.54mm_Vertical")
+    )
+    (path "/4cfee851-0cc5-4d3d-a57d-b2108e11a482"
+      (reference "DBG10") (unit 1) (value "TX") (footprint "Connector_PinSocket_2.54mm:PinSocket_1x01_P2.54mm_Vertical")
+    )
     (path "/0abfc9bc-cfd1-4238-99b4-f5788aa9a167"
-      (reference "DBG?") (unit 1) (value "RX") (footprint "Connector_PinSocket_2.54mm:PinSocket_1x01_P2.54mm_Vertical")
-    )
-    (path "/1a72f5d6-44ee-46ae-8a18-fbbb82588964"
-      (reference "DBG?") (unit 1) (value "5V") (footprint "Connector_PinSocket_2.54mm:PinSocket_1x01_P2.54mm_Vertical")
-    )
-    (path "/4cfee851-0cc5-4d3d-a57d-b2108e11a482"
-      (reference "DBG?") (unit 1) (value "TX") (footprint "Connector_PinSocket_2.54mm:PinSocket_1x01_P2.54mm_Vertical")
-    )
-    (path "/5c744d00-6e74-484c-b63b-3b58dd05dd79"
-      (reference "DBG?") (unit 1) (value "GND") (footprint "Connector_PinSocket_2.54mm:PinSocket_1x01_P2.54mm_Vertical")
+      (reference "DBG11") (unit 1) (value "RX") (footprint "Connector_PinSocket_2.54mm:PinSocket_1x01_P2.54mm_Vertical")
     )
     (path "/f9587540-9e33-42f9-8e4e-2bbaf53fb241"
-      (reference "DBG?") (unit 1) (value "RTS") (footprint "Connector_PinSocket_2.54mm:PinSocket_1x01_P2.54mm_Vertical")
-    )
-    (path "/feeb044e-58ef-4711-90fe-4a14fad0b279"
-      (reference "DBG?") (unit 1) (value "CTS") (footprint "Connector_PinSocket_2.54mm:PinSocket_1x01_P2.54mm_Vertical")
+      (reference "DBG12") (unit 1) (value "RTS") (footprint "Connector_PinSocket_2.54mm:PinSocket_1x01_P2.54mm_Vertical")
     )
     (path "/b0c15786-e0b2-4699-9893-07fcd4088d87"

Commit message: ordered version
Parts:
- removed DBG1, DBG7: GND, Connector_PinSocket_2.54mm:PinSocket_1x01_P2.54mm_Vertical, symbol Connector:TestPoint
- removed DBG10, DBG4: TX, Connector_PinSocket_2.54mm:PinSocket_1x01_P2.54mm_Vertical, symbol Connector:TestPoint
- removed DBG11, DBG5: RX, Connector_PinSocket_2.54mm:PinSocket_1x01_P2.54mm_Vertical, symbol Connector:TestPoint
- removed DBG12, DBG6: RTS, Connector_PinSocket_2.54mm:PinSocket_1x01_P2.54mm_Vertical, symbol Connector:TestPoint
- removed DBG2, DBG8: CTS, Connector_PinSocket_2.54mm:PinSocket_1x01_P2.54mm_Vertical, symbol Connector:TestPoint
- removed DBG3, DBG9: 5V, Connector_PinSocket_2.54mm:PinSocket_1x01_P2.54mm_Vertical, symbol Connector:TestPoint
- removed J1, J2: Conn_ARM_SWD_TagConnect_TC2030-NL, Connector:Tag-Connect_TC2030-IDC-NL_2x03_P1.27mm_Vertical, symbol Connector:Conn_ARM_SWD_TagConnect_TC2030-NL
- added U3, U4: SWD_Connector_3pin, entropy:SM03B-SRSS-TB, symbol entropy:SWD_Connector_3pin
- added U5: Debug_UART_l, entropy:Header_6pin, symbol entropy:Header_6pin
- added U6: Debug_UART_r, entropy:Header_6pin, symbol entropy:Header_6pin
Connections:
- net dbg_uart_rx_l: now also U5.5
- net dbg_uart_rx_r: now also U6.5
- net dbg_uart_tx_l: now also U5.4
- net dbg_uart_tx_r: now also U6.4
- net gnd_l: now also U3.2 (GND), U5.1
- net gnd_r: now also U4.2 (GND), U6.1
- net swclk_l: now also U3.1 (SCK)
- net swclk_r: now also U4.1 (SCK)
- net swdio_l: now also U3.3 (SIO)
- net swdio_r: now also U4.3 (SIO)
- net vcc_l: now also U5.2
- net vcc_r: now also U6.2
