File: pcb/corneds.kicad_pcb (KiCad board)
At the start: 2 copper layers, 309.4 x 105.8 mm, 126 parts, among them J3 AudioJack4, J4 AudioJack4, SW1 SW_Push, SW10 SW_Push, SW11 SW_Push, SW12 SW_Push, SW13 SW_Push, SW14 SW_Push, SW15 SW_Push, SW16 SW_Push, SW17 SW_Push, SW18 SW_Push, SW19 SW_Push, SW2 SW_Push, SW20 SW_Push, SW21 SW_Push, SW22 SW_Push, SW23 SW_Push, SW24 SW_Push, SW25 SW_Push, SW26 SW_Push, SW27 SW_Push, SW28 SW_Push, SW29 SW_Push, SW3 SW_Push, SW30 SW_Push, SW31 SW_Push, SW32 SW_Push, SW33 SW_Push, SW34 SW_Push, SW35 SW_Push, SW36 SW_Push, SW37 SW_Push, SW38 SW_Push, SW39 SW_Push, SW4 SW_Push, SW40 SW_Push, SW41 SW_Push, SW42 SW_Push, SW5 SW_Push, SW6 SW_Push, SW7 SW_Push, SW8 SW_Push, SW9 SW_Push, U1 Pico, U2 Pico, U3 SWD_Connector_3pin, U4 SWD_Connector_3pin, U5 Debug_UART_l, U6 Debug_UART_r

Commit message: right side is working but left side needs pins updated
Routing:
- net /dbg_uart_tx_l: track 109.2 -> 101.2 mm, vias 1 -> 0
- net /row2_l: track 189.0 -> 181.6 mm
- net /row3_l: track 149.5 -> 142.1 mm
- net /dbg_uart_rx_l: track 111.0 -> 103.9 mm
Other:
- board text added: "06 Dec 2023"
- board text added: "66 Dec 2023"
- board text removed: "26 Nov 2023"

Commit message: fixed silk
Other:
- board text removed: "66 Dec 2023"
Changed lines of the file:
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@@
     (effects (font (size 1.5 1.5) (thickness 0.3)) (justify mirror))
   )
-  (gr_text "66 Dec 2023" (at 109.982 131.064) (layer "B.SilkS")
+  (gr_text "06 Dec 2023" (at 109.982 131.064) (layer "B.SilkS")
     (effects (font (size 1.5 1.5) (thickness 0.3)) (justify mirror))
   )
